File: Relay-Board.kicad_pcb (KiCad board)
At the start: 2 copper layers, 2 parts, among them U1 WEMOS_D1_mini, U9 WEMOS_Relay

Commit message: 2026-01-29
Parts:
- removed U9: WEMOS_Relay, RF_Module:WEMOS_D1_mini_light
- added J1: Screw_Terminal_01x10, TerminalBlock:TerminalBlock_Xinya_XY308-2.54-10P_1x10_P2.54mm_Horizontal, F.Cu at (66.0, 50.8)
- added J2: Screw_Terminal_01x02, TerminalBlock_CUI:TerminalBlock_CUI_TB007-508-02_1x02_P5.08mm_Horizontal, F.Cu at (22.9, 30.5)
- added J4: Screw_Terminal_01x10, TerminalBlock_CUI:TerminalBlock_CUI_TB007-508-10_1x10_P5.08mm_Horizontal, F.Cu at (81.2, 63.5)
- added J5: Screw_Terminal_01x02, TerminalBlock:TerminalBlock_Xinya_XY308-2.54-2P_1x02_P2.54mm_Horizontal, F.Cu at (20.3, 48.3)
- moved U1 15.1 mm to (33.0, 25.4), turned to 0 degrees
Connections:
- U1 pad 11: Net-(J1-Pin_6) -> /_D4
- U1 pad 12: Net-(J1-Pin_5) -> /_D3
- U1 pad 13: Net-(J1-Pin_4) -> /_D2
- U1 pad 14: Net-(J1-Pin_3) -> /_D1
- U1 pad 3: unconnected-(U1-D0-Pad3) -> /_D0
- U1 pad 4: Net-(J1-Pin_7) -> /_D5
- U1 pad 5: Net-(J1-Pin_8) -> /_D6
- U1 pad 6: Net-(J1-Pin_9) -> /_D7
- U1 pad 7: Net-(U1-CS/D8) -> unconnected-(U1-CS/D8-Pad7)
Routing:
- net Net-(J1-Pin_1): track 0.00 -> 111.7 mm
- net Net-(J1-Pin_2): track 0.00 -> 97.7 mm
- net /_D0: track 0.00 -> 76.1 mm
- net /_D5: track 0.00 -> 68.2 mm
- net /_D6: track 0.00 -> 65.7 mm
- net /_D7: track 0.00 -> 64.0 mm
- net /_D1: track 0.00 -> 35.3 mm
- net /_D2: track 0.00 -> 31.9 mm
- net /_D3: track 0.00 -> 29.7 mm
- net /_D4: track 0.00 -> 27.5 mm

Commit message: 2026-01-30
Parts:
- added H1: MountingHole, MountingHole:MountingHole_3.2mm_M3, F.Cu at (11.8, 5.08)
- added H2: MountingHole, MountingHole:MountingHole_3.2mm_M3, F.Cu at (87.2, 78.0)
- added H3: MountingHole, MountingHole:MountingHole_3.2mm_M3, F.Cu at (87.2, 5.08)
- added H4: MountingHole, MountingHole:MountingHole_3.2mm_M3, F.Cu at (11.8, 78.0)
- moved J2 7.18 mm to (17.8, 25.4), turned to -90 degrees
Routing:
- net /_D0: track 76.1 -> 65.4 mm
- net Net-(J1-Pin_2): track 97.7 -> 107.7 mm
- net /_D1: track 35.3 -> 30.7 mm
- net /_D7: track 64.0 -> 68.3 mm
- net /_D5: track 68.2 -> 65.7 mm
- net /_D2: track 31.9 -> 29.6 mm
- net Net-(J1-Pin_1): track 111.7 -> 110.0 mm
- net /_D6: track 65.7 -> 66.5 mm
Other:
- board text added: "1"
- board text added: "10"
- board text added: "2"
- board text added: "3"
- board text added: "3V3"
- board text added: "4"
- board text added: "5"
- board text added: "5V"
- board text added: "5VDC"
- board text added: "6"
- board text added: "7"
- board text added: "8"
- board text added: "9"
- board text added: "A0"
- board text added: "D0"
- board text added: "D1"
- board text added: "D2"
- board text added: "D3"
- board text added: "D4"
- board text added: "D5"
- board text added: "D6"
- board text added: "D7"
- board text added: "D8"
- board text added: "GND"
- board text added: "RST"
- board text added: "RX"
- board text added: "TX"
