File: Relay-Board.kicad_sch (KiCad schematic)
At the start: 3 parts, among them J1 Conn_01x10_Pin, U1 WEMOS_D1_mini, U9 WEMOS_Relay

Commit message: 2026-01-29
Parts:
- removed J1: Conn_01x10_Pin, symbol Connector:Conn_01x10_Pin
- removed U9: WEMOS_Relay, RF_Module:WEMOS_D1_mini_light, symbol New_Library:WEMOS_Relay
- added J1: Screw_Terminal_01x10, TerminalBlock:TerminalBlock_Xinya_XY308-2.54-10P_1x10_P2.54mm_Horizontal, symbol Connector:Screw_Terminal_01x10
- added J2: Screw_Terminal_01x02, TerminalBlock_CUI:TerminalBlock_CUI_TB007-508-02_1x02_P5.08mm_Horizontal, symbol Connector:Screw_Terminal_01x02
- added J4: Screw_Terminal_01x10, TerminalBlock_CUI:TerminalBlock_CUI_TB007-508-10_1x10_P5.08mm_Horizontal, symbol Connector:Screw_Terminal_01x10
- added J5: Screw_Terminal_01x02, TerminalBlock:TerminalBlock_Xinya_XY308-2.54-2P_1x02_P2.54mm_Horizontal, symbol Connector:Screw_Terminal_01x02
Connections:
- net at U1.10 (GND): now also J1.2 (Pin_2), J2.1 (Pin_1), J4.2 (Pin_2), J5.1 (Pin_1)
- net _D4: now reaches U1.11 (D4)
- net _D4: now also J1.7 (Pin_7), J4.7 (Pin_7)
- net _D3: now reaches U1.12 (D3)
- net _D3: now also J1.8 (Pin_8), J4.8 (Pin_8)
- net _D2: now reaches U1.13 (SDA/D2)
- net _D2: now also J1.9 (Pin_9), J4.9 (Pin_9)
- net _D1: now reaches U1.14 (SCL/D1)
- net _D1: now also J1.10 (Pin_10), J4.10 (Pin_10)
- net _D0: now reaches U1.3 (D0)
- net _D0: now also J1.6 (Pin_6), J4.6 (Pin_6)
- net _D5: now reaches U1.4 (SCK/D5)
- net _D5: now also J1.5 (Pin_5), J4.5 (Pin_5)
- net _D6: now reaches U1.5 (MISO/D6)
- net _D6: now also J1.4 (Pin_4), J4.4 (Pin_4)
- net _D7: now reaches U1.6 (MOSI/D7)
- net _D7: now also J1.3 (Pin_3), J4.3 (Pin_3)
- net at U1.9 (5V): now also J1.1 (Pin_1), J2.2 (Pin_2), J4.1 (Pin_1), J5.2 (Pin_2)

Commit message: 2026-01-30
Parts:
- added H1, H2, H3, H4: MountingHole, MountingHole:MountingHole_3.2mm_M3, symbol Mechanical:MountingHole
